Commit message: Add SO-ARM-101 robot description, launch files, and keyboard teleoperation scripts

File: so_arm_101_description/urdf/so_101.ros2_control.xacro (robot description, xacro)
@@ -8,31 +8,43 @@
     <joint name="base_link_to_link1">
       <command_interface name="position"/>
-      <state_interface name="position"/>
+      <state_interface name="position">
+        <param name="initial_value">0.0</param>
+      </state_interface>
       <state_interface name="velocity"/>
     </joint>
     <joint name="link1_to_link2">
       <command_interface name="position"/>
-      <state_interface name="position"/>
+      <state_interface name="position">
+        <param name="initial_value">-1.0</param>
+      </state_interface>
       <state_interface name="velocity"/>
     </joint>
     <joint name="link2_to_link3">
       <command_interface name="position"/>
-      <state_interface name="position"/>
+      <state_interface name="position">
+        <param name="initial_value">1.5</param>
+      </state_interface>
       <state_interface name="velocity"/>
     </joint>
     <joint name="link3_to_link4">
       <command_interface name="position"/>
-      <state_interface name="position"/>
+      <state_interface name="position">
+        <param name="initial_value">0.0</param>
+      </state_interface>
       <state_interface name="velocity"/>
     </joint>
     <joint name="link4_to_link5">
       <command_interface name="position"/>
-      <state_interface name="position"/>
+      <state_interface name="position">
+        <param name="initial_value">0.0</param>
+      </state_interface>
       <state_interface name="velocity"/>
     </joint>
-    <!-- Gripper joints (both clamps) -->
+    <!-- Only the physical actuator is commanded; left_clamp is a mimic. -->
     <joint name="right_clamp">
       <command_interface name="position"/>
-      <state_interface name="position"/>
+      <state_interface name="position">
+        <param name="initial_value">0.0</param>
+      </state_interface>
       <state_interface name="velocity"/>
     </joint>

File: so_arm_101_description/urdf/so_101.urdf.xacro (robot description, xacro)
@@ -185,5 +185,5 @@
     <child link="link1_1"/>
     <axis xyz="-0.0 -0.008727 0.999962"/>
-    <limit lower="-2.094395" upper="2.094395" effort="1.5" velocity="5.236"/>
+    <limit lower="-2.094395" upper="2.094395" effort="100.0" velocity="5.236"/>
     <dynamics damping="0.1" friction="0.05"/>
     <safety_controller soft_lower_limit="-2.044" soft_upper_limit="2.044" k_position="100" k_velocity="10"/>
@@ -195,5 +195,5 @@
     <child link="link2_1"/>
     <axis xyz="-0.999962 -0.008726 -7.6e-05"/>
-    <limit lower="-3.228859" upper="0.174533" effort="1.5" velocity="5.236"/>
+    <limit lower="-3.228859" upper="0.174533" effort="100.0" velocity="5.236"/>
     <dynamics damping="0.1" friction="0.05"/>
     <safety_controller soft_lower_limit="-3.179" soft_upper_limit="0.125" k_position="100" k_velocity="10"/>
@@ -205,5 +205,5 @@
     <child link="link3_1"/>
     <axis xyz="-0.999924 -0.00865 -0.008802"/>
-    <limit lower="0.0" upper="3.316126" effort="1.5" velocity="5.236"/>
+    <limit lower="0.0" upper="3.316126" effort="100.0" velocity="5.236"/>
     <dynamics damping="0.1" friction="0.05"/>
     <safety_controller soft_lower_limit="0.05" soft_upper_limit="3.266" k_position="100" k_velocity="10"/>
@@ -215,5 +215,5 @@
     <child link="link4_1"/>
     <axis xyz="-0.999848 0.000153 -0.017451"/>
-    <limit lower="-1.658063" upper="1.658063" effort="1.5" velocity="5.236"/>
+    <limit lower="-1.658063" upper="1.658063" effort="100.0" velocity="5.236"/>
     <dynamics damping="0.1" friction="0.05"/>
     <safety_controller soft_lower_limit="-1.608" soft_upper_limit="1.608" k_position="100" k_velocity="10"/>
@@ -225,5 +225,5 @@
     <child link="link5_1"/>
     <axis xyz="-1e-06 0.999961 0.008803"/>
-    <limit lower="-4.276057" upper="1.570796" effort="1.5" velocity="5.236"/>
+    <limit lower="-4.276057" upper="1.570796" effort="100.0" velocity="5.236"/>
     <dynamics damping="0.1" friction="0.05"/>
     <safety_controller soft_lower_limit="-4.226" soft_upper_limit="1.521" k_position="100" k_velocity="10"/>
@@ -235,8 +235,8 @@
     <child link="clamp_1"/>
     <axis xyz="0.999848 -0.000154 0.017451"/>
-    <limit lower="0.0" upper="0.037" effort="1.5" velocity="0.05"/>
-    <dynamics damping="0.5" friction="0.1"/>
-  </joint>
-  <!-- Gripper: left clamp (mimic of right_clamp, inverted) -->
+    <limit lower="0.0" upper="0.037" effort="1000.0" velocity="1.0"/>
+    <dynamics damping="0.01" friction="0.0"/>
+  </joint>
+  <!-- Passive side mechanically coupled to the single commanded joint. -->
   <joint name="left_clamp" type="prismatic">
     <origin xyz="0.072828 -0.222278 -0.183875" rpy="0 0 0"/>
@@ -244,6 +244,6 @@
     <child link="clamp_2"/>
     <axis xyz="0.999848 -0.000154 0.017451"/>
-    <limit lower="-0.038" upper="0.0" effort="1.5" velocity="0.05"/>
-    <dynamics damping="0.5" friction="0.1"/>
+    <limit lower="-0.037" upper="0.0" effort="1000.0" velocity="1.0"/>
+    <dynamics damping="0.01" friction="0.0"/>
     <mimic joint="right_clamp" multiplier="-1" offset="0"/>
   </joint>

Commit message: Enhance SO-ARM-101 robot description with improved .gitignore, VSCode settings, and updated README. Refine keyboard teleoperation for gradual gripper control and add tests for controller configuration and joint dynamics.

File: so_arm_101_description/urdf/so_101.ros2_control.xacro (robot description, xacro)
@@ -41,5 +41,9 @@
       <state_interface name="velocity"/>
     </joint>
-    <!-- Only the physical actuator is commanded; left_clamp is a mimic. -->
+    <!--
+      Only the physical actuator belongs to ros2_control.  Do not list the
+      passive finger here: gz_ros2_control would add a second velocity-based
+      mimic loop on top of Gazebo's native SDF mimic constraint.
+    -->
     <joint name="right_clamp">
       <command_interface name="position"/>
@@ -47,8 +51,4 @@
         <param name="initial_value">0.0</param>
       </state_interface>
-      <state_interface name="velocity"/>
-    </joint>
-    <joint name="left_clamp">
-      <state_interface name="position"/>
       <state_interface name="velocity"/>
     </joint>

File: so_arm_101_description/urdf/so_101.urdf.xacro (robot description, xacro)
@@ -235,5 +235,5 @@
     <child link="clamp_1"/>
     <axis xyz="0.999848 -0.000154 0.017451"/>
-    <limit lower="0.0" upper="0.037" effort="1000.0" velocity="1.0"/>
+    <limit lower="0.0" upper="0.037" effort="100.0" velocity="0.05"/>
     <dynamics damping="0.01" friction="0.0"/>
   </joint>
@@ -244,5 +244,5 @@
     <child link="clamp_2"/>
     <axis xyz="0.999848 -0.000154 0.017451"/>
-    <limit lower="-0.037" upper="0.0" effort="1000.0" velocity="1.0"/>
+    <limit lower="-0.037" upper="0.0" effort="100.0" velocity="0.05"/>
     <dynamics damping="0.01" friction="0.0"/>
     <mimic joint="right_clamp" multiplier="-1" offset="0"/>
