Commit message: Update SO-ARM-101 configurations and calibration parameters
- Adjust initial joint values for link1_to_link2 and link2_to_link3 to 0.0
- Refine joint limits and safety controller parameters for link1_to_link2 and link2_to_link3
- Modify gripper settings in so101_follower.json for improved control
- Add calibration file argument to real.launch.py and hardware_node.py
- Enhance lerobot_adapter.py with joint calibration logic for accurate motor control
- Update keyboard teleoperation limits to match new joint configurations

File: so_arm_101/so_arm_101_description/urdf/so_101.ros2_control.xacro (robot description, xacro)
@@ -17,5 +17,5 @@
       <command_interface name="position"/>
       <state_interface name="position">
-        <param name="initial_value">-1.0</param>
+        <param name="initial_value">0.0</param>
       </state_interface>
       <state_interface name="velocity"/>
@@ -24,5 +24,5 @@
       <command_interface name="position"/>
       <state_interface name="position">
-        <param name="initial_value">1.5</param>
+        <param name="initial_value">0.0</param>
       </state_interface>
       <state_interface name="velocity"/>

File: so_arm_101/so_arm_101_description/urdf/so_101.urdf.xacro (robot description, xacro)
@@ -193,21 +193,23 @@
   <!-- Joint 2: Shoulder pitch — STS3215 servo -->
   <joint name="link1_to_link2" type="revolute">
-    <origin xyz="0.020891 -0.031313 0.091377" rpy="0 0 0"/>
+    <!-- Rotate the joint frame so q=0 is the LeRobot calibration zero. -->
+    <origin xyz="0.020891 -0.031313 0.091377" rpy="1.57079632679 0 0"/>
     <parent link="link1_1"/>
     <child link="link2_1"/>
     <axis xyz="-0.999962 -0.008726 -7.6e-05"/>
-    <limit lower="-3.228859" upper="0.174533" effort="100.0" velocity="5.236"/>
-    <dynamics damping="0.1" friction="0.05"/>
-    <safety_controller soft_lower_limit="-3.179" soft_upper_limit="0.125" k_position="100" k_velocity="10"/>
+    <limit lower="-1.825" upper="1.825" effort="100.0" velocity="5.236"/>
+    <dynamics damping="0.1" friction="0.05"/>
+    <safety_controller soft_lower_limit="-1.775" soft_upper_limit="1.775" k_position="100" k_velocity="10"/>
   </joint>
   <!-- Joint 3: Elbow — STS3215 servo -->
   <joint name="link2_to_link3" type="revolute">
-    <origin xyz="0.00151 0.112435 0.029417" rpy="0 0 0"/>
+    <!-- Rotate the joint frame so q=0 is the LeRobot calibration zero. -->
+    <origin xyz="0.00151 0.112435 0.029417" rpy="-1.6 0 0"/>
     <parent link="link2_1"/>
     <child link="link3_1"/>
     <axis xyz="-0.999924 -0.00865 -0.008802"/>
-    <limit lower="0.0" upper="3.316126" effort="100.0" velocity="5.236"/>
-    <dynamics damping="0.1" friction="0.05"/>
-    <safety_controller soft_lower_limit="0.05" soft_upper_limit="3.266" k_position="100" k_velocity="10"/>
+    <limit lower="-1.71" upper="1.71" effort="100.0" velocity="5.236"/>
+    <dynamics damping="0.1" friction="0.05"/>
+    <safety_controller soft_lower_limit="-1.66" soft_upper_limit="1.66" k_position="100" k_velocity="10"/>
   </joint>
   <!-- Joint 4: Wrist pitch — STS3215 servo -->

Commit message: Refactor SO-ARM-101 hardware interface and driver integration
- Updated real.yaml configuration to allow dynamic port assignment and changed topic names for state and command.
- Introduced driver.launch.py to encapsulate the LeRobot driver node launch logic.
- Modified real.launch.py to include driver.launch.py for better modularity.
- Added package dependencies for so_arm_101_description and python3-yaml.
- Enhanced hardware_node.py to support new command and state topics, and improved joint state publishing with velocity.
- Implemented gripper calibration loading from a YAML file.
- Created unit tests for the lerobot_adapter to validate joint and gripper conversions.
- Established a new hardware interface package (so_arm_101_hardware_interface) with a SystemInterface implementation for ros2_control.
- Updated MoveIt configuration files to ensure compatibility with the new hardware interface.
- Added tests for MoveIt configuration validation.
- Refined keyboard teleoperation to utilize joint limits from the description package.

File: so_arm_101/so_arm_101_description/urdf/so_101.ros2_control.xacro (robot description, xacro)
@@ -1,55 +1,42 @@
 <?xml version="1.0" ?>
 <robot name="so_101" xmlns:xacro="http://www.ros.org/wiki/xacro">
-  <!-- The hardware interfaces are reusable; the Gazebo plugin is optional. -->
+  <!-- The block remains top-level so tooling can inspect the control joints. -->
   <ros2_control name="so_101_system" type="system">
     <hardware>
-      <plugin>gz_ros2_control/GazeboSimSystem</plugin>
+      <plugin>$(arg hardware_plugin)</plugin>
+      <xacro:if value="$(arg use_real_ros2_control)">
+        <param name="state_topic">/so101_hardware/raw_joint_states</param>
+        <param name="command_topic">/so101_hardware/command_positions</param>
+      </xacro:if>
     </hardware>
-    <!-- Arm joints -->
     <joint name="base_link_to_link1">
       <command_interface name="position"/>
-      <state_interface name="position">
-        <param name="initial_value">0.0</param>
-      </state_interface>
+      <state_interface name="position"><param name="initial_value">0.0</param></state_interface>
       <state_interface name="velocity"/>
     </joint>
     <joint name="link1_to_link2">
       <command_interface name="position"/>
-      <state_interface name="position">
-        <param name="initial_value">0.0</param>
-      </state_interface>
+      <state_interface name="position"><param name="initial_value">0.0</param></state_interface>
       <state_interface name="velocity"/>
     </joint>
     <joint name="link2_to_link3">
       <command_interface name="position"/>
-      <state_interface name="position">
-        <param name="initial_value">0.0</param>
-      </state_interface>
+      <state_interface name="position"><param name="initial_value">0.0</param></state_interface>
       <state_interface name="velocity"/>
     </joint>
     <joint name="link3_to_link4">
       <command_interface name="position"/>
-      <state_interface name="position">
-        <param name="initial_value">0.0</param>
-      </state_interface>
+      <state_interface name="position"><param name="initial_value">0.0</param></state_interface>
       <state_interface name="velocity"/>
     </joint>
     <joint name="link4_to_link5">
       <command_interface name="position"/>
-      <state_interface name="position">
-        <param name="initial_value">0.0</param>
-      </state_interface>
+      <state_interface name="position"><param name="initial_value">0.0</param></state_interface>
       <state_interface name="velocity"/>
     </joint>
-    <!--
-      Only the physical actuator belongs to ros2_control.  Do not list the
-      passive finger here: gz_ros2_control would add a second velocity-based
-      mimic loop on top of Gazebo's native SDF mimic constraint.
-    -->
+    <!-- Only the physical actuator is controlled; left_clamp is mimic. -->
     <joint name="right_clamp">
       <command_interface name="position"/>
-      <state_interface name="position">
-        <param name="initial_value">0.0</param>
-      </state_interface>
+      <state_interface name="position"><param name="initial_value">0.0</param></state_interface>
       <state_interface name="velocity"/>
     </joint>

File: so_arm_101/so_arm_101_description/urdf/so_101.urdf.xacro (robot description, xacro)
@@ -2,8 +2,11 @@
 <robot name="so_101" xmlns:xacro="http://www.ros.org/wiki/xacro">
   <xacro:arg name="use_gz_ros2_control" default="false"/>
+  <xacro:arg name="use_real_ros2_control" default="false"/>
   <xacro:arg name="controllers_file" default=""/>
+  <xacro:arg name="hardware_plugin" default="gz_ros2_control/GazeboSimSystem"/>
   <!-- Includes -->
   <xacro:include filename="$(find so_arm_101_description)/urdf/materials.xacro"/>
   <xacro:include filename="$(find so_arm_101_description)/urdf/so_101.ros2_control.xacro"/>
+  <xacro:property name="joint_limits" value="${xacro.load_yaml('$(find so_arm_101_description)/config/joint_limits.yaml')['joint_limits']}"/>
   <!-- ============================================================ -->
   <!-- World frame — fixes the robot base to the ground              -->
@@ -187,5 +190,5 @@
     <child link="link1_1"/>
     <axis xyz="-0.0 -0.008727 0.999962"/>
-    <limit lower="-2.094395" upper="2.094395" effort="100.0" velocity="5.236"/>
+    <limit lower="${joint_limits['base_link_to_link1']['min_position']}" upper="${joint_limits['base_link_to_link1']['max_position']}" effort="${joint_limits['base_link_to_link1']['max_effort']}" velocity="${joint_limits['base_link_to_link1']['max_velocity']}"/>
     <dynamics damping="0.1" friction="0.05"/>
     <safety_controller soft_lower_limit="-2.044" soft_upper_limit="2.044" k_position="100" k_velocity="10"/>
@@ -198,5 +201,5 @@
     <child link="link2_1"/>
     <axis xyz="-0.999962 -0.008726 -7.6e-05"/>
-    <limit lower="-1.825" upper="1.825" effort="100.0" velocity="5.236"/>
+    <limit lower="${joint_limits['link1_to_link2']['min_position']}" upper="${joint_limits['link1_to_link2']['max_position']}" effort="${joint_limits['link1_to_link2']['max_effort']}" velocity="${joint_limits['link1_to_link2']['max_velocity']}"/>
     <dynamics damping="0.1" friction="0.05"/>
     <safety_controller soft_lower_limit="-1.775" soft_upper_limit="1.775" k_position="100" k_velocity="10"/>
@@ -209,5 +212,5 @@
     <child link="link3_1"/>
     <axis xyz="-0.999924 -0.00865 -0.008802"/>
-    <limit lower="-1.71" upper="1.71" effort="100.0" velocity="5.236"/>
+    <limit lower="${joint_limits['link2_to_link3']['min_position']}" upper="${joint_limits['link2_to_link3']['max_position']}" effort="${joint_limits['link2_to_link3']['max_effort']}" velocity="${joint_limits['link2_to_link3']['max_velocity']}"/>
     <dynamics damping="0.1" friction="0.05"/>
     <safety_controller soft_lower_limit="-1.66" soft_upper_limit="1.66" k_position="100" k_velocity="10"/>
@@ -219,5 +222,5 @@
     <child link="link4_1"/>
     <axis xyz="-0.999848 0.000153 -0.017451"/>
-    <limit lower="-1.658063" upper="1.658063" effort="100.0" velocity="5.236"/>
+    <limit lower="${joint_limits['link3_to_link4']['min_position']}" upper="${joint_limits['link3_to_link4']['max_position']}" effort="${joint_limits['link3_to_link4']['max_effort']}" velocity="${joint_limits['link3_to_link4']['max_velocity']}"/>
     <dynamics damping="0.1" friction="0.05"/>
     <safety_controller soft_lower_limit="-1.608" soft_upper_limit="1.608" k_position="100" k_velocity="10"/>
@@ -229,5 +232,5 @@
     <child link="link5_1"/>
     <axis xyz="-1e-06 0.999961 0.008803"/>
-    <limit lower="-4.276057" upper="1.570796" effort="100.0" velocity="5.236"/>
+    <limit lower="${joint_limits['link4_to_link5']['min_position']}" upper="${joint_limits['link4_to_link5']['max_position']}" effort="${joint_limits['link4_to_link5']['max_effort']}" velocity="${joint_limits['link4_to_link5']['max_velocity']}"/>
     <dynamics damping="0.1" friction="0.05"/>
     <safety_controller soft_lower_limit="-4.226" soft_upper_limit="1.521" k_position="100" k_velocity="10"/>
@@ -239,5 +242,5 @@
     <child link="clamp_1"/>
     <axis xyz="0.999848 -0.000154 0.017451"/>
-    <limit lower="0.0" upper="0.037" effort="100.0" velocity="0.05"/>
+    <limit lower="${joint_limits['right_clamp']['min_position']}" upper="${joint_limits['right_clamp']['max_position']}" effort="${joint_limits['right_clamp']['max_effort']}" velocity="${joint_limits['right_clamp']['max_velocity']}"/>
     <dynamics damping="0.01" friction="0.0"/>
   </joint>
@@ -248,5 +251,5 @@
     <child link="clamp_2"/>
     <axis xyz="0.999848 -0.000154 0.017451"/>
-    <limit lower="-0.037" upper="0.0" effort="100.0" velocity="0.05"/>
+    <limit lower="${joint_limits['left_clamp']['min_position']}" upper="${joint_limits['left_clamp']['max_position']}" effort="${joint_limits['left_clamp']['max_effort']}" velocity="${joint_limits['left_clamp']['max_velocity']}"/>
     <dynamics damping="0.01" friction="0.0"/>
     <mimic joint="right_clamp" multiplier="-1" offset="0"/>
