Commit message: Add Tool Center Point visualization and update kinematics configuration for SO-ARM-101

File: so_arm_101/so_arm_101_description/urdf/materials.xacro (robot description, xacro)
@@ -4,3 +4,7 @@
     <color rgba="0.700 0.700 0.700 1.000"/>
   </material>
+  <!-- Marcador visual do Tool Center Point no RViz. -->
+  <material name="tcp_marker">
+    <color rgba="1.000 0.050 0.050 1.000"/>
+  </material>
 </robot>

File: so_arm_101/so_arm_101_description/urdf/so_101.urdf.xacro (robot description, xacro)
@@ -141,4 +141,20 @@
     </collision>
   </link>
+  <!-- Tool Center Point: centro nominal de pega entre os dedos. -->
+  <link name="gripper_tcp">
+    <!-- Esfera vermelha para localizar o TCP no RobotModel do RViz. -->
+    <visual>
+      <geometry>
+        <sphere radius="0.006"/>
+      </geometry>
+      <material name="tcp_marker"/>
+    </visual>
+  </link>
+  <joint name="link5_to_gripper_tcp" type="fixed">
+    <parent link="link5_1"/>
+    <child link="gripper_tcp"/>
+    <!-- Os dedos ocupam aproximadamente y=-0.052 a -0.132 m em link5_1. -->
+    <origin xyz="0 -0.10 0" rpy="0 0 0"/>
+  </joint>
   <link name="clamp_1">
     <inertial>

Commit message: Add laptop camera module and update URDF configuration for improved visualization

File: so_arm_101/so_arm_101_description/urdf/materials.xacro (robot description, xacro)
@@ -8,3 +8,10 @@
     <color rgba="1.000 0.050 0.050 1.000"/>
   </material>
+  <!-- Materiais da webcam compacta fixada no punho. -->
+  <material name="camera_body">
+    <color rgba="0.075 0.075 0.085 1.000"/>
+  </material>
+  <material name="camera_lens">
+    <color rgba="0.020 0.120 0.180 1.000"/>
+  </material>
 </robot>

File: so_arm_101/so_arm_101_description/urdf/so_101.urdf.xacro (robot description, xacro)
@@ -7,4 +7,5 @@
   <!-- Includes -->
   <xacro:include filename="$(find so_arm_101_description)/urdf/materials.xacro"/>
+  <xacro:include filename="$(find so_arm_101_description)/urdf/laptop_camera.xacro"/>
   <xacro:include filename="$(find so_arm_101_description)/urdf/so_101.ros2_control.xacro"/>
   <xacro:property name="joint_limits" value="${xacro.load_yaml('$(find so_arm_101_description)/config/joint_limits.yaml')['joint_limits']}"/>
@@ -157,4 +158,6 @@
     <origin xyz="0 -0.13 0" rpy="0 0 0"/>
   </joint>
+  <!-- Webcam modular colada à face inferior do link4_1. -->
+  <xacro:laptop_camera parent_link="link4_1"/>
   <link name="clamp_1">
     <inertial>
