Commit message: Add AprilTag detection package with launch configuration, detector node, and URDF integration

File: so_arm_101/so_arm_101_description/urdf/laptop_camera.xacro (robot description, xacro)
@@ -30,4 +30,11 @@
       <origin xyz="-0.01 -0.04 -0.016" rpy="1.57079632679 0 0"/>
     </joint>
+    <!-- ROS optical-frame convention: X right, Y down, Z forward (lens). -->
+    <link name="${camera_link}_optical_frame"/>
+    <joint name="${camera_link}_to_optical_frame" type="fixed">
+      <parent link="${camera_link}"/>
+      <child link="${camera_link}_optical_frame"/>
+      <origin xyz="0 0 0" rpy="-1.57079632679 0 3.14159265359"/>
+    </joint>
   </xacro:macro>
 </robot>

Commit message: Update laptop camera dimensions for improved accuracy in URDF representation

File: so_arm_101/so_arm_101_description/urdf/laptop_camera.xacro (robot description, xacro)
@@ -11,5 +11,5 @@
       <visual>
         <geometry>
-          <box size="0.050 0.002 0.015"/>
+          <box size="0.0635 0.0026 0.0087"/>
         </geometry>
         <material name="camera_body"/>
