Commit message: feat(lidar): implement ROS 2 node for LiDAR XV-11 driver
- Added lidar_node.py to handle LiDAR data acquisition and publishing.
- Created package.xml for lidar package dependencies and metadata.
- Implemented setup.py and setup.cfg for package installation.
- Added test cases for lidar driver and node functionality.
- Included resource files for package sharing.

feat(robot_description): add robot description and configuration

- Created CMakeLists.txt and package.xml for robot_description package.
- Added URDF and configuration files for robot structure.
- Implemented tests for URDF structure and parameter validation.

refactor(so_arm_101): update package references and structure

- Changed package references from cbr_* to generic names.
- Updated README and test files to reflect new package structure.
- Refactored URDF files to use new naming conventions for components.

File: so_arm_101/so_arm_101_description/urdf/camera_mount.xacro (robot description, xacro)
@@ -2,5 +2,5 @@
 <robot xmlns:xacro="http://www.ros.org/wiki/xacro">
   <!-- Camera rigidly mounted under link4_1. Measurements are lens-centered. -->
-  <xacro:macro name="cbr_camera_mount" params="parent_link">
+  <xacro:macro name="camera_mount" params="parent_link">
     <link name="camera_link">
       <visual>

File: so_arm_101/so_arm_101_description/urdf/so_101.urdf.xacro (robot description, xacro)
@@ -26,5 +26,5 @@
   </xacro:unless>
   <xacro:if value="${attach_to_mobile_base}">
-    <xacro:property name="arm_mount" value="${xacro.load_yaml('$(find cbr_robot_description)/config/arm_mount.yaml')['arm_mount']}"/>
+    <xacro:property name="arm_mount" value="${xacro.load_yaml('$(find robot_description)/config/arm_mount.yaml')['arm_mount']}"/>
     <joint name="mobile_base_to_arm" type="fixed">
       <parent link="upper_platform_link"/>
@@ -174,5 +174,5 @@
   </joint>
   <!-- Camera measured and rigidly mounted to the underside of link4_1. -->
-  <xacro:cbr_camera_mount parent_link="link4_1"/>
+  <xacro:camera_mount parent_link="link4_1"/>
   <link name="clamp_1">
     <inertial>
