Commit message: Update joint positions and object coordinates for improved pick-and-place functionality in SO-ARM-101

File: so_arm_101/so_arm_101_description/urdf/so_101.urdf.xacro (robot description, xacro)
@@ -155,5 +155,5 @@
     <child link="gripper_tcp"/>
     <!-- Os dedos ocupam aproximadamente y=-0.052 a -0.132 m em link5_1. -->
-    <origin xyz="0 -0.10 0" rpy="0 0 0"/>
+    <origin xyz="0 -0.127 0" rpy="0 0 0"/>
   </joint>
   <link name="clamp_1">
@@ -224,5 +224,5 @@
   <joint name="link2_to_link3" type="revolute">
     <!-- Rotate the joint frame so q=0 is the LeRobot calibration zero. -->
-    <origin xyz="0.00151 0.112435 0.029417" rpy="-1.6 0 0"/>
+    <origin xyz="0.00151 0.112435 0.029417" rpy="-1.7 0 0"/>
     <parent link="link2_1"/>
     <child link="link3_1"/>

Commit message: Refactor pick-and-place functionality by updating joint positions, adding new group states, and restructuring code for improved clarity and maintainability.

File: so_arm_101/so_arm_101_description/urdf/so_101.urdf.xacro (robot description, xacro)
@@ -155,5 +155,5 @@
     <child link="gripper_tcp"/>
     <!-- Os dedos ocupam aproximadamente y=-0.052 a -0.132 m em link5_1. -->
-    <origin xyz="0 -0.127 0" rpy="0 0 0"/>
+    <origin xyz="0 -0.13 0" rpy="0 0 0"/>
   </joint>
   <link name="clamp_1">

Commit message: Update joint limits, adjust follower configurations, and refine object handling in pegar_e_colocar script

File: so_arm_101/so_arm_101_description/urdf/so_101.urdf.xacro (robot description, xacro)
@@ -247,5 +247,5 @@
   <!-- Joint 5: Wrist roll — STS3215 servo -->
   <joint name="link4_to_link5" type="revolute">
-    <origin xyz="-0.01732 -0.060045 -0.000831" rpy="0 0 0"/>
+    <origin xyz="-0.01732 -0.060045 -0.000831" rpy="0 -1.5707963267 0"/>
     <parent link="link4_1"/>
     <child link="link5_1"/>

Commit message: feat: update robot configuration and description

File: so_arm_101/so_arm_101_description/urdf/so_101.urdf.xacro (robot description, xacro)
@@ -146,5 +146,5 @@
       <origin xyz="-0.007062 0.120627 -0.152066" rpy="0 0 0"/>
       <geometry>
-        <mesh filename="package://so_arm_101_description/meshes/visual/link5_1.stl" scale="0.001 0.001 0.001"/>
+        <mesh filename="package://so_arm_101_description/meshes/visual/link5_1.stl" scale="1 1 1"/>
       </geometry>
       <material name="silver"/>
@@ -153,5 +153,5 @@
       <origin xyz="-0.007062 0.120627 -0.152066" rpy="0 0 0"/>
       <geometry>
-        <mesh filename="package://so_arm_101_description/meshes/collision/link5_1.stl" scale="0.001 0.001 0.001"/>
+        <mesh filename="package://so_arm_101_description/meshes/collision/link5_1.stl" scale="1 1 1"/>
       </geometry>
     </collision>
@@ -170,6 +170,5 @@
     <parent link="link5_1"/>
     <child link="gripper_tcp"/>
-    <!-- Os dedos ocupam aproximadamente y=-0.052 a -0.132 m em link5_1. -->
-    <origin xyz="0 -0.13 0" rpy="0 0 0"/>
+    <origin xyz="0 -0.10 0" rpy="0 0 0"/>
   </joint>
   <!-- Camera measured and rigidly mounted to the underside of link4_1. -->
@@ -177,19 +176,19 @@
   <link name="clamp_1">
     <inertial>
-      <origin xyz="0.0601695113719365 0.14480677890200364 0.1844826866723634" rpy="0 0 0"/>
+      <origin xyz="0 0 0" rpy="0 0 0"/>
       <mass value="0.15381179772652928"/>
       <inertia ixx="8.6e-05" iyy="4.1e-05" izz="7.3e-05" ixy="-1e-06" iyz="4e-06" ixz="-2e-06"/>
     </inertial>
     <visual>
-      <origin xyz="0.045072 0.340704 0.033971" rpy="0 0 0"/>
-      <geometry>
-        <mesh filename="package://so_arm_101_description/meshes/visual/clamp_1.stl" scale="0.001 0.001 0.001"/>
-      </geometry>
-      <material name="silver"/>
-    </visual>
-    <collision>
-      <origin xyz="0.045072 0.340704 0.033971" rpy="0 0 0"/>
-      <geometry>
-        <mesh filename="package://so_arm_101_description/meshes/visual/clamp_1.stl" scale="0.001 0.001 0.001"/>
+      <origin xyz="0 0 0" rpy="1.57079632679 1.57079632679 0"/>
+      <geometry>
+        <mesh filename="package://so_arm_101_description/meshes/visual/pinca.stl" scale="1 1 1"/>
+      </geometry>
+      <material name="silver"/>
+    </visual>
+    <collision>
+      <origin xyz="0 0 0" rpy="0 0 0"/>
+      <geometry>
+        <mesh filename="package://so_arm_101_description/meshes/visual/pinca.stl" scale="1 1 1"/>
       </geometry>
     </collision>
@@ -197,19 +196,19 @@
   <link name="clamp_2">
     <inertial>
-      <origin xyz="-0.0800042161303889 0.1470101120878245 0.18506826370370444" rpy="0 0 0"/>
+      <origin xyz="0 0 0" rpy="0 0 0"/>
       <mass value="0.15381179772652928"/>
       <inertia ixx="8.6e-05" iyy="4.1e-05" izz="7.3e-05" ixy="1e-06" iyz="-4e-06" ixz="-2e-06"/>
     </inertial>
     <visual>
-      <origin xyz="-0.07989 0.342905 0.031809" rpy="0 0 0"/>
-      <geometry>
-        <mesh filename="package://so_arm_101_description/meshes/visual/clamp_2.stl" scale="0.001 0.001 0.001"/>
-      </geometry>
-      <material name="silver"/>
-    </visual>
-    <collision>
-      <origin xyz="-0.07989 0.342905 0.031809" rpy="0 0 0"/>
-      <geometry>
-        <mesh filename="package://so_arm_101_description/meshes/visual/clamp_2.stl" scale="0.001 0.001 0.001"/>
+      <origin xyz="0 0 0" rpy="1.57079632679 -1.57079632679 0"/>
+      <geometry>
+        <mesh filename="package://so_arm_101_description/meshes/visual/pinca.stl" scale="1 1 1"/>
+      </geometry>
+      <material name="silver"/>
+    </visual>
+    <collision>
+      <origin xyz="0 0 0" rpy="0 0 0"/>
+      <geometry>
+        <mesh filename="package://so_arm_101_description/meshes/visual/pinca.stl" scale="1 1 1"/>
       </geometry>
     </collision>
@@ -272,5 +271,5 @@
   <!-- Gripper: right clamp (primary) — STS3215 servo -->
   <joint name="right_clamp" type="prismatic">
-    <origin xyz="-0.052134 -0.220077 -0.186037" rpy="0 0 0"/>
+    <origin xyz="0.005 -0.065 0" rpy="0 0 0"/>
     <parent link="link5_1"/>
     <child link="clamp_1"/>
@@ -281,5 +280,5 @@
   <!-- Passive side mechanically coupled to the single commanded joint. -->
   <joint name="left_clamp" type="prismatic">
-    <origin xyz="0.072828 -0.222278 -0.183875" rpy="0 0 0"/>
+    <origin xyz="-0.005 -0.065 0" rpy="0 0 0"/>
     <parent link="link5_1"/>
     <child link="clamp_2"/>

Commit message: fix: adjust parameters for controller server and recovery search positions

File: so_arm_101/so_arm_101_description/urdf/so_101.urdf.xacro (robot description, xacro)
@@ -170,5 +170,5 @@
     <parent link="link5_1"/>
     <child link="gripper_tcp"/>
-    <origin xyz="0 -0.10 0" rpy="0 0 0"/>
+    <origin xyz="0 -0.12 0" rpy="0 0 0"/>
   </joint>
   <!-- Camera measured and rigidly mounted to the underside of link4_1. -->

Commit message: Refactor code structure for improved readability and maintainability; removed redundant code blocks and optimized functions.

File: so_arm_101/so_arm_101_description/urdf/so_101.urdf.xacro (robot description, xacro)
@@ -146,5 +146,5 @@
       <origin xyz="-0.007062 0.120627 -0.152066" rpy="0 0 0"/>
       <geometry>
-        <mesh filename="package://so_arm_101_description/meshes/visual/link5_1.stl" scale="1 1 1"/>
+        <mesh filename="package://so_arm_101_description/meshes/visual/link5_1.stl" scale="0.001 0.001 0.001"/>
       </geometry>
       <material name="silver"/>
@@ -153,5 +153,5 @@
       <origin xyz="-0.007062 0.120627 -0.152066" rpy="0 0 0"/>
       <geometry>
-        <mesh filename="package://so_arm_101_description/meshes/collision/link5_1.stl" scale="1 1 1"/>
+        <mesh filename="package://so_arm_101_description/meshes/collision/link5_1.stl" scale="0.001 0.001 0.001"/>
       </geometry>
     </collision>

Commit message: feat: adicionar tópico de alvo de liberação de contêiner e atualizar a lógica de publicação no servidor de manipulação

File: so_arm_101/so_arm_101_description/urdf/so_101.urdf.xacro (robot description, xacro)
@@ -170,5 +170,5 @@
     <parent link="link5_1"/>
     <child link="gripper_tcp"/>
-    <origin xyz="0 -0.12 0" rpy="0 0 0"/>
+    <origin xyz="0 -0.08 0" rpy="0 0 0"/>
   </joint>
   <!-- Camera measured and rigidly mounted to the underside of link4_1. -->

Commit message: feat: ajustar incertezas de detecção e melhorar lógica de posicionamento na mesa

File: so_arm_101/so_arm_101_description/urdf/so_101.urdf.xacro (robot description, xacro)
@@ -170,5 +170,5 @@
     <parent link="link5_1"/>
     <child link="gripper_tcp"/>
-    <origin xyz="0 -0.08 0" rpy="0 0 0"/>
+    <origin xyz="0 -0.12 0" rpy="0 0 0"/>
   </joint>
   <!-- Camera measured and rigidly mounted to the underside of link4_1. -->

Commit message: feat: ajustar limites de área mínima de contornos para melhorar a detecção de objetos

File: so_arm_101/so_arm_101_description/urdf/so_101.urdf.xacro (robot description, xacro)
@@ -170,5 +170,5 @@
     <parent link="link5_1"/>
     <child link="gripper_tcp"/>
-    <origin xyz="0 -0.12 0" rpy="0 0 0"/>
+    <origin xyz="0 -0.06 0" rpy="0 0 0"/>
   </joint>
   <!-- Camera measured and rigidly mounted to the underside of link4_1. -->

Commit message: feat: ajustar parâmetros de geometria do contêiner e adicionar teste para ignorar cubos da mesma cor

File: so_arm_101/so_arm_101_description/urdf/so_101.urdf.xacro (robot description, xacro)
@@ -170,5 +170,5 @@
     <parent link="link5_1"/>
     <child link="gripper_tcp"/>
-    <origin xyz="0 -0.06 0" rpy="0 0 0"/>
+    <origin xyz="0 -0.12 0" rpy="0 0 0"/>
   </joint>
   <!-- Camera measured and rigidly mounted to the underside of link4_1. -->

Commit message: feat: adicionar suporte para visualização de tabela de depuração e ajustar restrições de posição do TCP

File: so_arm_101/so_arm_101_description/urdf/so_101.urdf.xacro (robot description, xacro)
@@ -170,5 +170,18 @@
     <parent link="link5_1"/>
     <child link="gripper_tcp"/>
-    <origin xyz="0 -0.08 0" rpy="0 0 0"/>
+    <origin xyz="0 -0.12 0" rpy="0 0 0"/>
+  </joint>
+  <link name="gripper_tcp_near">
+    <visual>
+      <geometry>
+        <sphere radius="0.006"/>
+      </geometry>
+      <material name="tcp_marker"/>
+    </visual>
+  </link>
+  <joint name="link5_to_gripper_tcp_near" type="fixed">
+    <parent link="link5_1"/>
+    <child link="gripper_tcp_near"/>
+    <origin xyz="0 -0.07 0" rpy="0 0 0"/>
   </joint>
   <!-- Camera measured and rigidly mounted to the underside of link4_1. -->

Commit message: feat: remover referência ao gripper_tcp_near e ajustar restrições de posição no código de manipulação

File: so_arm_101/so_arm_101_description/urdf/so_101.urdf.xacro (robot description, xacro)
@@ -170,18 +170,5 @@
     <parent link="link5_1"/>
     <child link="gripper_tcp"/>
-    <origin xyz="0 -0.12 0" rpy="0 0 0"/>
-  </joint>
-  <link name="gripper_tcp_near">
-    <visual>
-      <geometry>
-        <sphere radius="0.006"/>
-      </geometry>
-      <material name="tcp_marker"/>
-    </visual>
-  </link>
-  <joint name="link5_to_gripper_tcp_near" type="fixed">
-    <parent link="link5_1"/>
-    <child link="gripper_tcp_near"/>
-    <origin xyz="0 -0.07 0" rpy="0 0 0"/>
+    <origin xyz="0 -0.08 0" rpy="0 0 0"/>
   </joint>
   <!-- Camera measured and rigidly mounted to the underside of link4_1. -->

Commit message: feat: adicionar suporte para depósito em contêiner e ajustar configurações de movimento

File: so_arm_101/so_arm_101_description/urdf/so_101.urdf.xacro (robot description, xacro)
@@ -170,5 +170,19 @@
     <parent link="link5_1"/>
     <child link="gripper_tcp"/>
-    <origin xyz="0 -0.08 0" rpy="0 0 0"/>
+    <origin xyz="0 -0.12 0" rpy="0 0 0"/>
+  </joint>
+  <!-- TCP exclusivo para o depósito em contêiner. -->
+  <link name="gripper_tcp_near">
+    <visual>
+      <geometry>
+        <sphere radius="0.006"/>
+      </geometry>
+      <material name="tcp_marker"/>
+    </visual>
+  </link>
+  <joint name="link5_to_gripper_tcp_near" type="fixed">
+    <parent link="link5_1"/>
+    <child link="gripper_tcp_near"/>
+    <origin xyz="0 -0.09 0" rpy="0 0 0"/>
   </joint>
   <!-- Camera measured and rigidly mounted to the underside of link4_1. -->

Commit message: feat: ajustar lógica de depósito e referência de posição no robô

File: so_arm_101/so_arm_101_description/urdf/so_101.urdf.xacro (robot description, xacro)
@@ -184,5 +184,5 @@
     <parent link="link5_1"/>
     <child link="gripper_tcp_near"/>
-    <origin xyz="0 -0.09 0" rpy="0 0 0"/>
+    <origin xyz="0 -0.05 0" rpy="0 0 0"/>
   </joint>
   <!-- Camera measured and rigidly mounted to the underside of link4_1. -->

Commit message: adiciona keepout filter no mapa

File: so_arm_101/so_arm_101_description/urdf/so_101.urdf.xacro (robot description, xacro)
@@ -184,5 +184,5 @@
     <parent link="link5_1"/>
     <child link="gripper_tcp_near"/>
-    <origin xyz="0 -0.05 0" rpy="0 0 0"/>
+    <origin xyz="0 -0.07 0" rpy="0 0 0"/>
   </joint>
   <!-- Camera measured and rigidly mounted to the underside of link4_1. -->
