Commit message: feat: Enhance CBR robot bringup with unified controller management
- Updated `robot.launch.py` to integrate a single controller manager for both arm and base.
- Introduced `wait_for_hardware_states.py` to ensure complete feedback from arm and wheel joints before starting controllers.
- Added `controllers.yaml` configuration for managing joint states and controllers.
- Created `__init__.py` for package initialization and improved code organization.
- Implemented tests for controller configurations and URDF structure validation.
- Adjusted camera configuration to use the correct video device.
- Added new message type `WheelCommand` for better command handling.
- Updated deployment script to point to the correct robot IP.
- Enhanced robot description with a composed structure for the mobile base and arm.

File: cbr_base_description/urdf/cbr_base.urdf.xacro (robot description, xacro)
@@ -1,13 +1,6 @@
 <?xml version="1.0"?>
 <robot xmlns:xacro="http://www.ros.org/wiki/xacro" name="cbr_base">
-  <!-- Initial estimates. Replace them with measurements before physical tests.
-       Dimensions are in metres and masses are in kilograms. -->
-  <xacro:arg name="mock_hardware" default="true"/>
-  <xacro:arg name="serial_port" default="/dev/ttyUSB0"/>
-  <xacro:arg name="motor_ids" default="0,1,2,3"/>
-  <xacro:arg name="motor_directions" default="1,1,1,1"/>
-  <xacro:arg name="ticks_per_revolution" default="0"/>
-  <xacro:arg name="max_wheel_velocity" default="0"/>
-  <!-- Measurements to replace: wheels and their centre-to-centre spacing. -->
+  <!-- Validated physical dimensions in metres; masses are in kilograms. -->
+  <!-- Wheels and their measured centre-to-centre spacing. -->
   <xacro:property name="wheel_radius" value="0.034"/>
   <xacro:property name="wheel_width" value="0.034"/>
@@ -15,5 +8,5 @@
   <xacro:property name="track_width" value="0.275"/>
   <xacro:property name="wheel_mass" value="0.35"/>
-  <!-- Measurements to replace: hollow lower rectangular frame. -->
+  <!-- Hollow lower rectangular frame. -->
   <xacro:property name="lower_frame_length" value="0.232"/>
   <xacro:property name="lower_frame_width" value="0.232"/>
@@ -22,10 +15,10 @@
   <xacro:property name="lower_frame_ground_clearance" value="0.015"/>
   <xacro:property name="lower_frame_mass" value="6.0"/>
-  <!-- Measurements to replace: solid upper platform, larger than the frame. -->
+  <!-- Solid upper platform, larger than the frame. -->
   <xacro:property name="upper_platform_length" value="0.232"/>
   <xacro:property name="upper_platform_width" value="0.306"/>
   <xacro:property name="upper_platform_thickness" value="0.008"/>
   <xacro:property name="upper_platform_mass" value="2.0"/>
-  <!-- Measurements to replace: IMU box and pose relative to base_link. -->
+  <!-- IMU box and pose relative to base_link. -->
   <xacro:property name="imu_length" value="0.039"/>
   <xacro:property name="imu_width" value="0.020"/>
@@ -38,5 +31,5 @@
   <xacro:property name="imu_pitch" value="0.0"/>
   <xacro:property name="imu_yaw" value="-1.5708"/>
-  <!-- Measurements to replace: the single central orange/black LiDAR. -->
+  <!-- The single central orange/black LiDAR. -->
   <xacro:property name="lidar_body_length" value="0.078"/>
   <xacro:property name="lidar_body_width" value="0.078"/>
@@ -259,13 +252,8 @@
   <ros2_control name="CBRMecanumSystem" type="system">
     <hardware>
-      <plugin>cbr_base_hardware/MariolaSystem</plugin>
-      <param name="mock_hardware">$(arg mock_hardware)</param>
-      <param name="serial_port">$(arg serial_port)</param>
-      <param name="baud_rate">250000</param>
-      <param name="timeout_ms">10</param>
-      <param name="motor_ids">$(arg motor_ids)</param>
-      <param name="motor_directions">$(arg motor_directions)</param>
-      <param name="ticks_per_revolution">$(arg ticks_per_revolution)</param>
-      <param name="max_wheel_velocity">$(arg max_wheel_velocity)</param>
+      <plugin>cbr_base_hardware_interface/MariolaSystem</plugin>
+      <param name="state_topic">/cbr_base_hardware/raw_joint_states</param>
+      <param name="command_topic">/cbr_base_hardware/command_velocities</param>
+      <param name="state_timeout_sec">0.25</param>
     </hardware>
     <xacro:macro name="wheel_control" params="name">

File: so_arm_101/so_arm_101_description/urdf/so_101.urdf.xacro (robot description, xacro)
@@ -5,4 +5,6 @@
   <xacro:arg name="controllers_file" default=""/>
   <xacro:arg name="hardware_plugin" default="gz_ros2_control/GazeboSimSystem"/>
+  <xacro:arg name="arm_base_link_name" default="base_link"/>
+  <xacro:arg name="attach_to_mobile_base" default="false"/>
   <!-- Includes -->
   <xacro:include filename="$(find so_arm_101_description)/urdf/materials.xacro"/>
@@ -10,17 +12,30 @@
   <xacro:include filename="$(find so_arm_101_description)/urdf/so_101.ros2_control.xacro"/>
   <xacro:property name="joint_limits" value="${xacro.load_yaml('$(find so_arm_101_description)/config/joint_limits.yaml')['joint_limits']}"/>
+  <!-- Keep the complete arm reusable inside a larger robot description. -->
+  <xacro:macro name="so_101_arm" params="arm_base_link_name attach_to_mobile_base">
   <!-- ============================================================ -->
   <!-- World frame — fixes the robot base to the ground              -->
   <!-- ============================================================ -->
-  <link name="world"/>
-  <joint name="world_to_base" type="fixed">
-    <parent link="world"/>
-    <child link="base_link"/>
-    <origin xyz="0 0 0" rpy="0 0 0"/>
-  </joint>
+  <xacro:unless value="${attach_to_mobile_base}">
+    <link name="world"/>
+    <joint name="world_to_base" type="fixed">
+      <parent link="world"/>
+      <child link="${arm_base_link_name}"/>
+      <origin xyz="0 0 0" rpy="0 0 0"/>
+    </joint>
+  </xacro:unless>
+  <xacro:if value="${attach_to_mobile_base}">
+    <xacro:property name="arm_mount" value="${xacro.load_yaml('$(find cbr_robot_description)/config/arm_mount.yaml')['arm_mount']}"/>
+    <joint name="mobile_base_to_arm" type="fixed">
+      <parent link="upper_platform_link"/>
+      <child link="${arm_base_link_name}"/>
+      <origin xyz="${arm_mount['x']} ${arm_mount['y']} ${arm_mount['z']}"
+        rpy="${arm_mount['roll']} ${arm_mount['pitch']} ${arm_mount['yaw']}"/>
+    </joint>
+  </xacro:if>
   <!-- ============================================================ -->
   <!-- Links                                                         -->
   <!-- ============================================================ -->
-  <link name="base_link">
+  <link name="${arm_base_link_name}">
     <inertial>
       <origin xyz="-7.395983749131527e-05 0.018688778123587116 0.031975817456183726" rpy="0 0 0"/>
@@ -206,5 +221,5 @@
   <joint name="base_link_to_link1" type="revolute">
     <origin xyz="-9.9e-05 -0.007243 0.027983" rpy="0 0 0"/>
-    <parent link="base_link"/>
+    <parent link="${arm_base_link_name}"/>
     <child link="link1_1"/>
     <axis xyz="-0.0 -0.008727 0.999962"/>
@@ -274,3 +289,7 @@
     <mimic joint="right_clamp" multiplier="-1" offset="0"/>
   </joint>
+  </xacro:macro>
+  <xacro:so_101_arm
+    arm_base_link_name="$(arg arm_base_link_name)"
+    attach_to_mobile_base="$(arg attach_to_mobile_base)"/>
 </robot>

Commit message: feat: Implement ROS 2 IMU driver and configuration
- Added `imu_node.py` for publishing IMU data to ROS 2.
- Created configuration files for IMU and EKF parameters.
- Developed launch files for initializing the IMU and integrating with odometry.
- Implemented unit tests for IMU driver and message formatting.
- Updated package metadata and setup configuration for new dependencies.
- Enhanced error handling and logging in the IMU driver.
- Resolved calibration file paths dynamically in the hardware node.
- Ensured launch parameters can be overridden via command line.

File: cbr_base_description/urdf/cbr_base.urdf.xacro (robot description, xacro)
@@ -30,5 +30,6 @@
   <xacro:property name="imu_roll" value="0.0"/>
   <xacro:property name="imu_pitch" value="0.0"/>
-  <xacro:property name="imu_yaw" value="-1.5708"/>
+  <!-- O firmware já entrega X para frente, Y para esquerda e Z para cima. -->
+  <xacro:property name="imu_yaw" value="0.0"/>
   <!-- The single central orange/black LiDAR. -->
   <xacro:property name="lidar_body_length" value="0.078"/>

Commit message: feat: Add new launch file for physical arm and camera integration, update joint states for cube manipulation

File: cbr_base_description/urdf/cbr_base.urdf.xacro (robot description, xacro)
@@ -42,4 +42,7 @@
   <xacro:property name="lidar_center_y" value="0.0"/>
   <xacro:property name="lidar_center_height_above_ground" value="0.035"/>
+  <!-- Calibrado contra parede perpendicular: o zero físico do XV-11 estava
+       aproximadamente 11,5° à esquerda do eixo frontal da base. -->
+  <xacro:property name="lidar_yaw" value="-0.2007"/>
   <!-- Derived Z positions, relative to base_link at wheel-axle height. -->
   <xacro:property name="lower_bottom_z"
@@ -232,5 +235,5 @@
     <parent link="base_link"/><child link="lidar_front_link"/>
     <origin xyz="${lidar_center_x} ${lidar_center_y} ${lidar_center_height_above_ground - wheel_radius}"
-      rpy="0 0 0"/>
+      rpy="0 0 ${lidar_yaw}"/>
   </joint>
   <!-- Separate component link prevents RViz from reusing the orange material
