Commit message: Refactor SO-ARM-101 packages by removing unused launch files and scripts
- Deleted teleoperation launch file and associated dependencies.
- Removed unnecessary controller manager message dependency from package.xml.
- Cleaned up setup.py by removing unused entry points and launch files.
- Eliminated wait_for_controllers and wait_for_joint_states scripts to streamline the bringup process.
- Updated README.md to reflect changes in driver usage and configuration.
- Removed driver.launch.py and real.launch.py to simplify hardware launch process.
- Deleted MoveIt-related launch files to focus on essential configurations.
- Adjusted pegar_e_colocar.py to correct grasping angle calculations.
- Updated movimento.py to clarify server startup instructions.
- Removed test files related to launch profiles to maintain consistency with current configurations.

File: base_description/urdf/base.urdf.xacro (robot description, xacro)
@@ -239,5 +239,5 @@
   <!-- Separate component link prevents RViz from reusing the orange material
        on the black body. Both links still represent one physical LiDAR. -->
-  <link name="lidar_body_link">
+  <!-- <link name="lidar_body_link">
     <visual>
       <geometry><box size="${lidar_body_length} ${lidar_body_width} ${lidar_body_height}"/></geometry>
@@ -253,5 +253,5 @@
     <parent link="lidar_front_link"/><child link="lidar_body_link"/>
     <origin xyz="0 0 ${-(lidar_orange_height + lidar_body_height) / 2.0}"/>
-  </joint>
+  </joint> -->
   <ros2_control name="CBRMecanumSystem" type="system">
     <hardware>

Commit message: commit

File: base_description/urdf/base.urdf.xacro (robot description, xacro)
@@ -44,5 +44,5 @@
   <!-- Calibrado contra parede perpendicular: o zero físico do XV-11 estava
        aproximadamente 11,5° à esquerda do eixo frontal da base. -->
-  <xacro:property name="lidar_yaw" value="-0.2007"/>
+  <xacro:property name="lidar_yaw" value="-0.06"/>
   <!-- Derived Z positions, relative to base_link at wheel-axle height. -->
   <xacro:property name="lower_bottom_z"

Commit message: refactor: atualiza operacao do pacote vl53

File: base_description/urdf/base.urdf.xacro (robot description, xacro)
@@ -39,7 +39,7 @@
   <xacro:property name="lidar_orange_height" value="0.017"/>
   <xacro:property name="lidar_mass" value="0.12"/>
-  <xacro:property name="lidar_center_x" value="0.075"/>
+  <xacro:property name="lidar_center_x" value="0.002"/>
   <xacro:property name="lidar_center_y" value="0.0"/>
-  <xacro:property name="lidar_center_height_above_ground" value="0.035"/>
+  <xacro:property name="lidar_center_height_above_ground" value="0.07"/>
   <!-- Correção atual de montagem: aproximadamente 3,4° à esquerda do eixo
        frontal da base. -->

Commit message: fix: update reference timeout to 1.5 for base controller in multiple config files

File: base_description/urdf/base.urdf.xacro (robot description, xacro)
@@ -42,7 +42,10 @@
   <xacro:property name="lidar_center_y" value="0.0"/>
   <xacro:property name="lidar_center_height_above_ground" value="0.07"/>
+  <!-- O LiDAR está montado invertido: 180° em X preserva frente/trás e
+       troca direita/esquerda no plano da varredura. -->
+  <xacro:property name="lidar_roll" value="${pi}"/>
   <!-- Correção atual de montagem: aproximadamente 3,4° à esquerda do eixo
        frontal da base. -->
-  <xacro:property name="lidar_yaw" value="-0.06"/>
+  <xacro:property name="lidar_yaw" value="0.06"/>
   <!-- Derived Z positions, relative to base_link at wheel-axle height. -->
   <xacro:property name="lower_bottom_z"
@@ -235,5 +238,5 @@
     <parent link="base_link"/><child link="lidar_front_link"/>
     <origin xyz="${lidar_center_x} ${lidar_center_y} ${lidar_center_height_above_ground - wheel_radius}"
-      rpy="0 0 ${lidar_yaw}"/>
+      rpy="${lidar_roll} 0 ${lidar_yaw}"/>
   </joint>
   <!-- Separate component link prevents RViz from reusing the orange material

Commit message: feat: Enhance robot simulation capabilities and sensor integration
- Updated `comandos.txt` to ensure proper formatting for action goals.
- Modified `mission_manager.launch.py` to allow dynamic arena file configuration via launch arguments.
- Expanded `robot.urdf.xacro` to include Gazebo sensor configurations for LIDAR, IMU, and cameras.
- Added Gazebo model path to `package.xml` for `so_arm_101_description`.
- Enhanced `so_101.ros2_control.xacro` to support additional joint interfaces for simulation.
- Adjusted `so_101.urdf.xacro` to conditionally scale collision meshes based on simulation settings.
- Updated MoveIt configuration to support simulation parameters in `configuration.py`.
- Enhanced vision launch file to manage simulation parameters and camera settings dynamically.
- Refactored `VL53DistanceAction` to support simulated sensor pairs in Gazebo.
- Implemented `GazeboSensorPair` class to read simulated range sensors through ROS LaserScan.

File: base_description/urdf/base.urdf.xacro (robot description, xacro)
@@ -1,4 +1,4 @@
 <?xml version="1.0"?>
-<robot xmlns:xacro="http://www.ros.org/wiki/xacro" name="base">
+<robot xmlns:xacro="http://www.ros.org/wiki/xacro" xmlns:gz="http://gazebosim.org/schema" name="base">
   <!-- Validated physical dimensions in metres; masses are in kilograms. -->
   <!-- Wheels and their measured centre-to-centre spacing. -->
@@ -191,4 +191,22 @@
   <xacro:mecanum_wheel prefix="rear_left" x="${-wheelbase / 2.0}" y="${track_width / 2.0}"/>
   <xacro:mecanum_wheel prefix="rear_right" x="${-wheelbase / 2.0}" y="${-track_width / 2.0}"/>
+  <!-- Anisotropic 45 degree contact models the free rollers of each
+       mecanum wheel while ros2_control still drives the real four wheel joints. -->
+  <xacro:macro name="mecanum_contact" params="wheel direction_x direction_y">
+    <gazebo reference="${wheel}_wheel_link">
+      <collision>
+        <surface><friction><ode>
+          <mu>1.5</mu><mu2>0.02</mu2>
+          <fdir1 gz:expressed_in="base_footprint">${direction_x} ${direction_y} 0</fdir1>
+        </ode></friction></surface>
+      </collision>
+    </gazebo>
+  </xacro:macro>
+  <xacro:if value="$(arg use_gz_ros2_control)">
+    <xacro:mecanum_contact wheel="front_left" direction_x="1" direction_y="-1"/>
+    <xacro:mecanum_contact wheel="front_right" direction_x="1" direction_y="1"/>
+    <xacro:mecanum_contact wheel="rear_left" direction_x="1" direction_y="1"/>
+    <xacro:mecanum_contact wheel="rear_right" direction_x="1" direction_y="-1"/>
+  </xacro:if>
   <link name="imu_link">
     <visual>
@@ -259,12 +277,14 @@
   <ros2_control name="CBRMecanumSystem" type="system">
     <hardware>
-      <plugin>base_hardware_interface/MariolaSystem</plugin>
-      <param name="state_topic">/base_hardware/raw_joint_states</param>
-      <param name="command_topic">/base_hardware/command_velocities</param>
-      <param name="max_wheel_velocity_rad_s">11.0</param>
-      <!-- At 30 Hz, 0.50 s tolerates a short scheduling stall on the SBC.
-           Command freshness is guarded separately by the 0.30 s watchdog in
-           base_hardware, so this does not prolong a stale wheel command. -->
-      <param name="state_timeout_sec">1.50</param>
+      <xacro:if value="$(arg use_gz_ros2_control)">
+        <plugin>gz_ros2_control/GazeboSimSystem</plugin>
+      </xacro:if>
+      <xacro:unless value="$(arg use_gz_ros2_control)">
+        <plugin>base_hardware_interface/MariolaSystem</plugin>
+        <param name="state_topic">/base_hardware/raw_joint_states</param>
+        <param name="command_topic">/base_hardware/command_velocities</param>
+        <param name="max_wheel_velocity_rad_s">11.0</param>
+        <param name="state_timeout_sec">1.50</param>
+      </xacro:unless>
     </hardware>
     <xacro:macro name="wheel_control" params="name">

File: robot_description/urdf/robot.urdf.xacro (robot description, xacro)
@@ -1,4 +1,4 @@
 <?xml version="1.0"?>
-<robot xmlns:xacro="http://www.ros.org/wiki/xacro" name="robot">
+<robot xmlns:xacro="http://www.ros.org/wiki/xacro" xmlns:gz="http://gazebosim.org/schema" name="robot">
   <!-- These internal mode arguments are fixed by this composed description. -->
   <xacro:arg name="arm_base_link_name" default="arm_base_link"/>
@@ -10,3 +10,56 @@
   <xacro:include filename="$(find base_description)/urdf/base.urdf.xacro"/>
   <xacro:include filename="$(find so_arm_101_description)/urdf/so_101.urdf.xacro"/>
+  <!-- Gazebo sensors publish the same public topics as physical drivers. -->
+  <xacro:if value="$(arg use_gz_ros2_control)">
+    <gazebo reference="lidar_front_link">
+      <preserveFixedJoint>true</preserveFixedJoint>
+      <sensor name="front_lidar" type="gpu_lidar">
+        <always_on>true</always_on><update_rate>10</update_rate>
+        <topic>/scan_front</topic><gz_frame_id>lidar_front_link</gz_frame_id>
+        <lidar><scan><horizontal><samples>360</samples><resolution>1</resolution>
+          <min_angle>-${pi}</min_angle><max_angle>${pi}</max_angle>
+        </horizontal></scan><range><min>0.10</min><max>3.0</max><resolution>0.01</resolution></range></lidar>
+      </sensor>
+    </gazebo>
+    <gazebo reference="imu_link">
+      <preserveFixedJoint>true</preserveFixedJoint>
+      <sensor name="imu" type="imu">
+        <always_on>true</always_on><update_rate>50</update_rate>
+        <topic>/imu/data</topic><gz_frame_id>imu_link</gz_frame_id>
+      </sensor>
+    </gazebo>
+    <!-- SDF cameras look along +X. The physical lens looks along -Y. -->
+    <gazebo reference="camera_link">
+      <preserveFixedJoint>true</preserveFixedJoint>
+      <sensor name="wrist_camera" type="camera">
+        <pose>0 0 0 0 0 -1.57079632679</pose>
+        <always_on>true</always_on><update_rate>15</update_rate>
+        <topic>/camera/image_rect</topic>
+        <gz_frame_id>camera_optical_frame</gz_frame_id>
+        <camera><horizontal_fov>1.047</horizontal_fov>
+          <image><width>640</width><height>480</height><format>R8G8B8</format></image>
+          <clip><near>0.02</near><far>3.0</far></clip>
+        </camera>
+      </sensor>
+    </gazebo>
+    <!-- Narrow range sensors are independent of the wide safety LiDAR. -->
+    <gazebo reference="base_link">
+      <sensor name="vl53_left" type="gpu_lidar">
+        <pose>0.116 0.080 -0.005 0 0 0</pose>
+        <always_on>true</always_on><update_rate>20</update_rate>
+        <topic>/vl53/left/scan</topic><gz_frame_id>base_link</gz_frame_id>
+        <lidar><scan><horizontal><samples>1</samples><min_angle>0</min_angle>
+          <max_angle>0</max_angle></horizontal></scan>
+          <range><min>0.02</min><max>2.0</max><resolution>0.001</resolution></range></lidar>
+      </sensor>
+      <sensor name="vl53_right" type="gpu_lidar">
+        <pose>0.116 -0.080 -0.005 0 0 0</pose>
+        <always_on>true</always_on><update_rate>20</update_rate>
+        <topic>/vl53/right/scan</topic><gz_frame_id>base_link</gz_frame_id>
+        <lidar><scan><horizontal><samples>1</samples><min_angle>0</min_angle>
+          <max_angle>0</max_angle></horizontal></scan>
+          <range><min>0.02</min><max>2.0</max><resolution>0.001</resolution></range></lidar>
+      </sensor>
+    </gazebo>
+  </xacro:if>
 </robot>

File: so_arm_101/so_arm_101_description/urdf/so_101.ros2_control.xacro (robot description, xacro)
@@ -41,4 +41,11 @@
       <state_interface name="velocity"/>
     </joint>
+    <xacro:if value="$(arg use_gz_ros2_control)">
+      <!-- Gazebo requires a state-only interface to drive the passive mimic. -->
+      <joint name="left_clamp">
+        <state_interface name="position"><param name="initial_value">0.0</param></state_interface>
+        <state_interface name="velocity"/>
+      </joint>
+    </xacro:if>
   </ros2_control>
   <xacro:if value="$(arg use_gz_ros2_control)">

File: so_arm_101/so_arm_101_description/urdf/so_101.urdf.xacro (robot description, xacro)
@@ -153,5 +153,11 @@
       <origin xyz="-0.007062 0.120627 -0.152066" rpy="0 0 0"/>
       <geometry>
-        <mesh filename="package://so_arm_101_description/meshes/collision/link5_1.stl" scale="1 1 1"/>
+        <!-- This collision STL is stored in millimeters; the visual STL is in meters. -->
+        <xacro:if value="$(arg use_gz_ros2_control)">
+          <mesh filename="package://so_arm_101_description/meshes/collision/link5_1.stl" scale="0.001 0.001 0.001"/>
+        </xacro:if>
+        <xacro:unless value="$(arg use_gz_ros2_control)">
+          <mesh filename="package://so_arm_101_description/meshes/collision/link5_1.stl" scale="1 1 1"/>
+        </xacro:unless>
       </geometry>
     </collision>
@@ -202,5 +208,10 @@
     </visual>
     <collision>
-      <origin xyz="0 0 0" rpy="0 0 0"/>
+      <xacro:if value="$(arg use_gz_ros2_control)">
+        <origin xyz="0 0 0" rpy="1.57079632679 1.57079632679 0"/>
+      </xacro:if>
+      <xacro:unless value="$(arg use_gz_ros2_control)">
+        <origin xyz="0 0 0" rpy="0 0 0"/>
+      </xacro:unless>
       <geometry>
         <mesh filename="package://so_arm_101_description/meshes/visual/pinca.stl" scale="1 1 1"/>
@@ -222,5 +233,10 @@
     </visual>
     <collision>
-      <origin xyz="0 0 0" rpy="0 0 0"/>
+      <xacro:if value="$(arg use_gz_ros2_control)">
+        <origin xyz="0 0 0" rpy="1.57079632679 -1.57079632679 0"/>
+      </xacro:if>
+      <xacro:unless value="$(arg use_gz_ros2_control)">
+        <origin xyz="0 0 0" rpy="0 0 0"/>
+      </xacro:unless>
       <geometry>
         <mesh filename="package://so_arm_101_description/meshes/visual/pinca.stl" scale="1 1 1"/>
